File: Laser_diode.sch (KiCad schematic (older format))
At the start: 0 parts

Commit message: Added laser diode, power stage, connecting block in progress
Parts:
- added C?: C, symbol Device:C
- added C? (x3): 100n, symbol Device:C
- added R? (x6): R, symbol Device:R
- added R?: 1k, symbol Device:R
- added RV? (x2): R_POT, symbol Device:R_POT
- added U?: TL072, symbol Lib:PLT5_520B
- added U? (x3): TL072, symbol Amplifier_Operational:TL072
- added U?: INA280A2, Package_TO_SOT_SMD:SOT-23-5, symbol Amplifier_Current:INA198
- added U?: TL071, symbol Amplifier_Operational:TL071
Connections:
- new net: R?.2, U?.2, U?.5 (-)
- new net: C?.2, R?.2, RV?.1, U?.2 (-), U?.3
- new net: C?.1, R?.1, R?.2, RV?.2, U?.1
- new net: R?.1, R?.2, RV?.1, U?.6 (-)
- new net: R?.2, U?.1
- new net: R?.2, R?.2, U?.2 (-)
- new net: R?.1, U?.3 (+)
- new net +5V: C?.1, C?.2, U?.7 (V+), U?.8 (V+)
- new net -5V: C?.1, U?.4 (V-)
- new net 0V: C?.2, C?.2, R?.1, U?.2 (GND), U?.3 (+), U?.4 (V-), U?.5 (+)
- new net 7V: C?.1, U?.3 (V+)
- new net I_mes: R?.1, U?.6
- new net In: R?.1, U?.4 (+)
- new net Out: U?.1
- new net PD_mes: R?.1, RV?.2, U?.7
- no-connect marks 0 -> 4
