File: Power_supply.sch (KiCad schematic (older format))
At the start: 51 parts

Commit message: Removed MC34063 added DC/DC module & +-5V LDO
Parts:
- removed C? (x4): 100u, Capacitor_THT:CP_Radial_D6.3mm_P2.50mm, symbol Device:CP
- removed C?: 220p, symbol Device:C
- removed C? (x5): 10u, symbol Device:C
- removed C?: 100n, symbol Device:C
- removed C?: 22u, symbol Device:CP
- removed D?: D_Schottky, symbol Device:D_Schottky
- removed HS?: Heatsink, symbol Mechanical:Heatsink
- removed L?: 82u, symbol Device:L
- removed L?: 6u8, symbol Device:L
- removed R?: 0R680, Resistor_SMD:R_2512_6332Metric_Pad1.40x3.35mm_HandSolder, symbol Device:R
- removed R?: 18k, symbol Device:R
- removed R?: 3.9k, symbol Device:R
- removed RV?: R_POT, symbol Device:R_POT
- removed U?: MC34063AD, Package_SO:SOIC-8_3.9x4.9mm_P1.27mm, symbol Lib:MC34063AD
- removed U?: LD1086DTTR, Package_TO_SOT_SMD:TO-252-2, symbol Regulator_Linear:LD1086DTTR
- added C? (x4): 1u, symbol Device:C
- added C? (x3): 10u, symbol Device:C
- added U?: PDME2-S12-D9-S, symbol Lib:PDME2-S12-D5-S
- added U?: TC595002ECBTR, symbol Regulator_Linear:LT1175-5_SOT223
- added U?: MCP1701AT-5002I/CB, Package_TO_SOT_SMD:SOT-23, symbol Regulator_Linear:MCP1700-1202E_SOT23
Connections:
- net labels added: +5V, +9V, -5V, -9V, 5V_D, 7V_A
- net labels removed: -7V, 5V
- wire segments 199 -> 174
Other:
- note removed: "Zmienić Vout - aby pasowało do LDO"
- moved on the sheet: C?, U?

Commit message: Added PIDs blocks
Parts:
- added L?: L, symbol Device:L
Connections:
- net GND: now also L?.1
- net 0V: now reaches C?.1, C?.2, U?.5 (0V)
- net 0V: now also L?.2
Changed lines of the file:
@@
 L power:-5V #PWR?
 U 1 1 61B17643
-P 10850 1375
-F 0 "#PWR?" H 10850 1475 50  0001 C CNN
-F 1 "-5V" H 10865 1548 50  0000 C CNN
-F 2 "" H 10850 1375 50  0001 C CNN
-F 3 "" H 10850 1375 50  0001 C CNN
-	1    10850 1375
+P 10850 1525
+F 0 "#PWR?" H 10850 1625 50  0001 C CNN
+F 1 "-5V" H 10865 1698 50  0000 C CNN
+F 2 "" H 10850 1525 50  0001 C CNN
+F 3 "" H 10850 1525 50  0001 C CNN
+	1    10850 1525
 	-1   0    0    1
 $EndComp
@@
 Text HLabel 10975 1225 2    50   Output ~ 0
 +5V
-Text HLabel 10975 1325 2    50   Output ~ 0
+Text HLabel 10975 1475 2    50   Output ~ 0
 -5V
 Wire Wire Line
-	10850 1325 10975 1325
+	10850 1475 10975 1475
 Wire Wire Line
 	10850 1225 10975 1225
 Wire Wire Line
-	10850 1375 10850 1325
+	10850 1525 10850 1475
 Wire Wire Line
 	10850 1225 10850 1175
@@
 Wire Wire Line
 	4275 3550 4400 3550
+$Comp
+L Device:L L?
+U 1 1 61BD524D
+P 4525 4950
+F 0 "L?" V 4715 4950 50  0000 C CNN
+F 1 "L" V 4624 4950 50  0000 C CNN
+F 2 "" H 4525 4950 50  0001 C CNN
+F 3 "~" H 4525 4950 50  0001 C CNN
+	1    4525 4950
+	0    -1   -1   0
+$EndComp
+$Comp
+L power:GND #PWR?
+U 1 1 61BD572F
+P 4325 5050
+F 0 "#PWR?" H 4325 4800 50  0001 C CNN
+F 1 "GND" H 4330 4877 50  0000 C CNN
+F 2 "" H 4325 5050 50  0001 C CNN
+F 3 "" H 4325 5050 50  0001 C CNN
+	1    4325 5050
+	1    0    0    -1
+$EndComp
+Wire Wire Line
+	4325 5050 4325 4950
+Wire Wire Line
+	4325 4950 4375 4950
+Text Label 2750 3550 2    50   ~ 0
+0V
+Wire Wire Line
+	2600 3550 2750 3550
+Text Label 4800 4950 2    50   ~ 0
+0V
+Wire Wire Line
+	4800 4950 4675 4950
+Text Label 10850 1350 0    50   ~ 0
+0V
+Text HLabel 10975 1350 2    50   Output ~ 0
+0V
+Wire Wire Line
+	10975 1350 10850 1350
 $EndSCHEMATC

Commit message: Added laser diode, power stage, connecting block in progress
Changed lines of the file:
@@
 $Descr A4 11693 8268
 encoding utf-8
-Sheet 5 12
+Sheet 5 11
 Title ""
 Date ""
@@
 Wire Wire Line
 	850  900  850  1000
-Text Label 10775 875  0    50   ~ 0
-V_ld
 Text HLabel 10975 575  2    50   Output ~ 0
 7V
@@
 Text HLabel 10975 775  2    50   Output ~ 0
 3v3
-Text HLabel 10975 875  2    50   Output ~ 0
-V_LD
-Wire Wire Line
-	10775 875  10975 875
 Wire Wire Line
 	10975 775  10775 775
