File: Switch.sch (KiCad schematic (older format))
At the start: 4 parts

Commit message: Added integrator reset, fixed Switch.sch
Connections:
- net +5V: now also K?.A1; no longer K?.A2
- net at D?.1 (K), Q?.3 (C): now also K?.A2; no longer K?.A1
- net IN renamed OUT
Other:
- moved on the sheet: K?
Changed lines of the file:
@@
 F 3 "" H 4650 2400 50  0001 C CNN
 	1    4650 2400
-	0    1    1    0
+	0    -1   1    0
 $EndComp
 $Comp
@@
 	0    1    1    0
 $EndComp
-Text HLabel 9750 725  2    50   Output ~ 0
+Text HLabel 750  1325 0    50   Input ~ 0
 NC
-Text HLabel 9750 900  2    50   Output ~ 0
+Text HLabel 750  1150 0    50   Input ~ 0
 NO
-Text HLabel 750  1250 0    50   Input ~ 0
-IN
+Text HLabel 9750 1000 2    50   Output ~ 0
+OUT
 Text HLabel 750  750  0    50   Input ~ 0
 5V
@@
 	-1   0    0    -1
 $EndComp
-Text Label 5100 2500 2    50   ~ 0
+Text Label 4225 2500 0    50   ~ 0
 NC
-Text Label 5100 2700 2    50   ~ 0
+Text Label 4225 2700 0    50   ~ 0
 NO
-Wire Wire Line
-	5100 2700 4950 2700
-Wire Wire Line
-	4950 2500 5100 2500
-Text Label 9550 725  0    50   ~ 0
+Text Label 950  1325 2    50   ~ 0
 NC
-Text Label 9550 900  0    50   ~ 0
+Text Label 950  1150 2    50   ~ 0
 NO
-Text Label 900  1250 2    50   ~ 0
-In
-Wire Wire Line
-	900  1250 750  1250
-Text Label 4200 2600 0    50   ~ 0
-In
 $Comp
 L power:GND #PWR?
@@
 	6000 2525 5950 2525
 Wire Wire Line
-	4200 2600 4350 2600
-Wire Wire Line
 	6450 2525 6300 2525
 Wire Wire Line
-	9550 900  9750 900
+	950  1150 750  1150
 Wire Wire Line
-	9750 725  9550 725
+	750  1325 950  1325
+Wire Wire Line
+	4225 2700 4350 2700
+Wire Wire Line
+	4225 2500 4350 2500
+Text Label 9550 1000 0    50   ~ 0
+OUT
+Wire Wire Line
+	9550 1000 9750 1000
+Text Label 5150 2600 2    50   ~ 0
+OUT
+Wire Wire Line
+	5150 2600 4950 2600
 $EndSCHEMATC
